Commit message: Fingertip motion replay script completed - now we can now where the fingertips are wrt the camera

File: models/allegro_hand_description/urdf/model_new_connected.urdf (robot description, URDF)
Before this commit: robot allegrokinova, 30 links, 29 joints
Links:
- link kinova_link_1: geometry collision mesh filename=package://kinova_description/meshes/shoulder.STL; visual mesh filename=package://kinova_description/meshes/ring_big.STL
- link kinova_link_2: geometry collision mesh filename=package://kinova_description/meshes/arm.STL; visual mesh filename=package://kinova_description/meshes/arm.STL
- link kinova_link_3: geometry collision mesh filename=package://kinova_description/meshes/forearm.STL; visual mesh filename=package://kinova_description/meshes/forearm.STL
- link kinova_link_4: geometry collision mesh filename=package://kinova_description/meshes/wrist_spherical_1.STL; visual mesh filename=package://kinova_description/meshes/ring_small.STL
- link kinova_link_5: geometry collision mesh filename=package://kinova_description/meshes/wrist_spherical_2.STL; visual mesh filename=package://kinova_description/meshes/ring_small.STL
- link kinova_link_6: geometry collision mesh filename=package://kinova_description/meshes/hand_3finger.STL; visual mesh filename=package://kinova_description/meshes/hand_3finger.STL
- link kinova_link_base: geometry collision mesh filename=package://kinova_description/meshes/base.STL; visual mesh filename=package://kinova_description/meshes/base.STL

File: models/allegro_hand_description/urdf/model_new_final.urdf (robot description, URDF)
Before this commit: robot allegrokinova, 29 links, 28 joints
Links:
- link kinova_link_1: geometry collision mesh filename=package://kinova_description/meshes/shoulder.STL; visual mesh filename=package://kinova_description/meshes/ring_big.obj
- link kinova_link_2: geometry collision mesh filename=package://kinova_description/meshes/arm.STL; visual mesh filename=package://kinova_description/meshes/arm.obj
- link kinova_link_3: geometry collision mesh filename=package://kinova_description/meshes/forearm.STL; visual mesh filename=package://kinova_description/meshes/forearm.obj
- link kinova_link_4: geometry collision mesh filename=package://kinova_description/meshes/wrist_spherical_1.STL; visual mesh filename=package://kinova_description/meshes/ring_small.obj
- link kinova_link_5: geometry collision mesh filename=package://kinova_description/meshes/wrist_spherical_2.STL; visual mesh filename=package://kinova_description/meshes/ring_small.obj
- link kinova_link_base: geometry collision mesh filename=package://kinova_description/meshes/base.STL; visual mesh filename=package://kinova_description/meshes/base.obj
